Commit message: create 2 joint

File: CreateURDF/my_robot.urdf (robot description, URDF)
Before this commit: robot my_robot, 2 links, 1 joints
Links:
- added link third_link; visual box size=0.1 0.1 0.1
Joints:
- added joint second_third_joint: type fixed, parent second_link, child third_link, origin xyz=0 0 0.2 rpy=0 0 0

Commit message: fix different type of joint

File: CreateURDF/my_robot.urdf (robot description, URDF)
Before this commit: robot my_robot, 3 links, 2 joints
Links:
- removed link third_link
Joints:
- removed joint second_third_joint
- joint base_second_joint: axis (none) -> 1 0 0; limit (none) -> lower=-1.57 upper=0.5 effort=100 velocity=100; type fixed -> prismatic
