Commit message: complete robot

File: CreateURDF/robot-wheel.urdf (robot description, URDF)
Before this commit: robot my_robot, 2 links, 1 joints
Links:
- added link base_footprint
- added link caster_wheel_link; visual sphere radius=0.05
- added link left_wheel_link; visual cylinder length=0.05 radius=0.1
Joints:
- added joint base_caster_wheel_joint: type fixed, parent base_link, child caster_wheel_link, origin xyz=0.2 0 -0.05 rpy=0 0 0
- added joint base_footprint_joint: type fixed, parent base_footprint, child base_link, origin xyz=0 0 0.1 rpy=0 0 0
- added joint base_left_wheel_joint: type continuous, parent base_link, child left_wheel_link, origin xyz=-0.15 0.225 0 rpy=0 0 0, axis 0 1 0
