Commit message: fix xacro variable

File: ros2_ws/src/my_robot-description/urdf/robot-wheel.urdf.xacro (robot description, xacro)
@@ -1,4 +1,5 @@
 <?xml version="1.0" ?>
 <robot name="my_robot" xmlns:xacro="http://www.ros.org/wiki/xacro">
+    <xacro:property name="base_length" value="0.6"/>
     <material name="blue">
         <color rgba="1 0 0.6 1"/>
@@ -10,5 +11,5 @@
         <visual>
             <geometry>
-                <box size="0.6 0.4 0.2"/>
+                <box size="${base_length} 0.4 0.2"/>
             </geometry>
             <origin xyz="0 0 0.1" rpy="0 0 0" />
@@ -21,5 +22,5 @@
                 <cylinder radius="0.1" length="0.05"/>
             </geometry>
-            <origin xyz="0 0 0" rpy="1.57 0 0"/>
+            <origin xyz="0 0 0" rpy="${pi / 2.0} 0 0"/>
             <material name="grey"/>
         </visual>
@@ -30,5 +31,5 @@
                 <cylinder radius="0.1" length="0.05"/>
             </geometry>
-            <origin xyz="0 0 0" rpy="-1.57 0 0"/>
+            <origin xyz="0 0 0" rpy="${pi / 2.0} 0 0"/>
             <material name="grey"/>
         </visual>
@@ -51,5 +52,5 @@
         <parent link="base_link"/>
         <child link="right_wheel_link"/>
-        <origin xyz="-0.15 -0.225 0" rpy="0 0 0"/>
+        <origin xyz="${-base_length / 4.0} -0.225 0" rpy="0 0 0"/>
         <axis xyz="0 1 0"/>
     </joint>
@@ -57,5 +58,5 @@
         <parent link="base_link"/>
         <child link="left_wheel_link"/>
-        <origin xyz="-0.15 0.225 0" rpy="0 0 0"/>
+        <origin xyz="${-base_length / 4.0} 0.225 0" rpy="0 0 0"/>
         <axis xyz="0 1 0"/>
     </joint>
@@ -63,5 +64,5 @@
         <parent link="base_link"/>
         <child link="caster_wheel_link"/>
-        <origin xyz="0.2 0 -0.05" rpy="0 0 0"/>
+        <origin xyz="${base_length / 3.0} 0 -0.05" rpy="0 0 0"/>
     </joint>
     <joint name="base_footprint_joint" type="fixed">

Commit message: fix xacro functions

File: ros2_ws/src/my_robot-description/urdf/robot-wheel.urdf.xacro (robot description, xacro)
@@ -2,4 +2,8 @@
 <robot name="my_robot" xmlns:xacro="http://www.ros.org/wiki/xacro">
     <xacro:property name="base_length" value="0.6"/>
+    <xacro:property name="base_width" value="0.4"/>
+    <xacro:property name="base_height" value="0.2"/>
+    <xacro:property name="wheel_radius" value="0.1"/>
+    <xacro:property name="wheel_length" value="0.05"/>
     <material name="blue">
         <color rgba="1 0 0.6 1"/>
@@ -11,14 +15,27 @@
         <visual>
             <geometry>
-                <box size="${base_length} 0.4 0.2"/>
+                <box size="${base_length} ${base_width} ${base_height}"/>
             </geometry>
-            <origin xyz="0 0 0.1" rpy="0 0 0" />
+            <origin xyz="0 0 ${base_height / 2.0}" rpy="0 0 0" />
             <material name="blue"/>
         </visual>
     </link>
+    <!-- <xacro:macro name="Wheel_link" params="prefix">
+        <link name="${prefix}_wheel_link">
+            <visual>
+                <geometry>
+                    <cylinder radius="${wheel_radius}" length="${wheel_length}"/>
+                </geometry>
+                <origin xyz="0 0 0" rpy="${pi / 2.0} 0 0"/>
+                <material name="grey"/>
+            </visual>
+        </link>
+    </xacro:macro>
+    <xacro:Wheel_link prefix="right" />
+    <xacro:Wheel_link prefix="left" /> -->
     <link name="right_wheel_link">
         <visual>
             <geometry>
-                <cylinder radius="0.1" length="0.05"/>
+                <cylinder radius="${wheel_radius}" length="${wheel_length}"/>
             </geometry>
             <origin xyz="0 0 0" rpy="${pi / 2.0} 0 0"/>
@@ -29,5 +46,5 @@
         <visual>
             <geometry>
-                <cylinder radius="0.1" length="0.05"/>
+                <cylinder radius="${wheel_radius}" length="${wheel_length}"/>
             </geometry>
             <origin xyz="0 0 0" rpy="${pi / 2.0} 0 0"/>
@@ -38,5 +55,5 @@
         <visual>
             <geometry>
-                <sphere radius="0.05" />
+                <sphere radius="${wheel_radius/2.0}" />
             </geometry>
             <origin xyz="0 0 0" rpy="0 0 0"/>
@@ -52,5 +69,5 @@
         <parent link="base_link"/>
         <child link="right_wheel_link"/>
-        <origin xyz="${-base_length / 4.0} -0.225 0" rpy="0 0 0"/>
+        <origin xyz="${-base_length / 4.0} ${-(base_width+ wheel_length)/2.0} 0" rpy="0 0 0"/>
         <axis xyz="0 1 0"/>
     </joint>
@@ -58,5 +75,5 @@
         <parent link="base_link"/>
         <child link="left_wheel_link"/>
-        <origin xyz="${-base_length / 4.0} 0.225 0" rpy="0 0 0"/>
+        <origin xyz="${-base_length / 4.0} ${-(base_width+ wheel_length)/2.0} 0" rpy="0 0 0"/>
         <axis xyz="0 1 0"/>
     </joint>
@@ -64,10 +81,10 @@
         <parent link="base_link"/>
         <child link="caster_wheel_link"/>
-        <origin xyz="${base_length / 3.0} 0 -0.05" rpy="0 0 0"/>
+        <origin xyz="${base_length / 3.0} 0 ${-(base_height / 4)}" rpy="0 0 0"/>
     </joint>
     <joint name="base_footprint_joint" type="fixed">
         <parent link="base_footprint"/>
         <child link="base_link"/>
-        <origin xyz="0 0 0.1" rpy="0 0 0"/>
+        <origin xyz="0 0 ${base_height / 2.0}" rpy="0 0 0"/>
     </joint>
 </robot>

Commit message: fix xacro

File: ros2_ws/src/my_robot-description/urdf/robot-wheel.urdf.xacro (robot description, xacro)
@@ -1,90 +1,64 @@
 <?xml version="1.0" ?>
 <robot name="my_robot" xmlns:xacro="http://www.ros.org/wiki/xacro">
-    <xacro:property name="base_length" value="0.6"/>
-    <xacro:property name="base_width" value="0.4"/>
-    <xacro:property name="base_height" value="0.2"/>
-    <xacro:property name="wheel_radius" value="0.1"/>
-    <xacro:property name="wheel_length" value="0.05"/>
-    <material name="blue">
-        <color rgba="1 0 0.6 1"/>
-    </material>
-    <material name="grey">
-        <color rgba="0.5 0.5 0.5 1"/>
-    </material>
+    <xacro:include filename="common_properties.xacro" />
+    <xacro:property name="base_length" value="0.6" />
+    <xacro:property name="base_width" value="0.4" />
+    <xacro:property name="base_height" value="0.2" />
+    <xacro:property name="wheel_radius" value="0.1" />
+    <xacro:property name="wheel_length" value="0.05" />
+    <link name="base_footprint" />
     <link name="base_link">
         <visual>
             <geometry>
-                <box size="${base_length} ${base_width} ${base_height}"/>
+                <box size="${base_length} ${base_width} ${base_height}" />
             </geometry>
             <origin xyz="0 0 ${base_height / 2.0}" rpy="0 0 0" />
-            <material name="blue"/>
+            <material name="blue" />
         </visual>
+        <xacro:box-inertia m="5" l="${base_length}" w="${base_width}" h="${base_height}" xyz="0 0 ${base_height / 2.0}" rpy="0 0 0" />
     </link>
-    <!-- <xacro:macro name="Wheel_link" params="prefix">
+    <xacro:macro name="wheel_link" params="prefix">
         <link name="${prefix}_wheel_link">
             <visual>
                 <geometry>
-                    <cylinder radius="${wheel_radius}" length="${wheel_length}"/>
+                    <cylinder radius="${wheel_radius}" length="${wheel_length}" />
                 </geometry>
-                <origin xyz="0 0 0" rpy="${pi / 2.0} 0 0"/>
-                <material name="grey"/>
+                <origin xyz="0 0 0" rpy="${pi / 2.0} 0 0" />
+                <material name="grey" />
             </visual>
         </link>
     </xacro:macro>
-    <xacro:Wheel_link prefix="right" />
-    <xacro:Wheel_link prefix="left" /> -->
-    <link name="right_wheel_link">
-        <visual>
-            <geometry>
-                <cylinder radius="${wheel_radius}" length="${wheel_length}"/>
-            </geometry>
-            <origin xyz="0 0 0" rpy="${pi / 2.0} 0 0"/>
-            <material name="grey"/>
-        </visual>
-    </link>
-    <link name="left_wheel_link">
-        <visual>
-            <geometry>
-                <cylinder radius="${wheel_radius}" length="${wheel_length}"/>
-            </geometry>
-            <origin xyz="0 0 0" rpy="${pi / 2.0} 0 0"/>
-            <material name="grey"/>
-        </visual>
-    </link>
+    <xacro:wheel_link prefix="right" />
+    <xacro:wheel_link prefix="left" />
     <link name="caster_wheel_link">
         <visual>
             <geometry>
-                <sphere radius="${wheel_radius/2.0}" />
+                <sphere radius="${wheel_radius / 2.0}" />
             </geometry>
-            <origin xyz="0 0 0" rpy="0 0 0"/>
-            <material name="grey"/>
+            <origin xyz="0 0 0" rpy="0 0 0" />
+            <material name="grey" />
         </visual>
     </link>
-    <link name="base_footprint">
-        <visual>
-            <origin xyz="0 0 0" rpy="0 0 0"/>
-        </visual>
-    </link>
+    <joint name="base_joint" type="fixed">
+        <parent link="base_footprint" />
+        <child link="base_link" />
+        <origin xyz="0 0 ${wheel_radius}" rpy="0 0 0"/>
+    </joint>
     <joint name="base_right_wheel_joint" type="continuous">
-        <parent link="base_link"/>
-        <child link="right_wheel_link"/>
-        <origin xyz="${-base_length / 4.0} ${-(base_width+ wheel_length)/2.0} 0" rpy="0 0 0"/>
-        <axis xyz="0 1 0"/>
+        <parent link="base_link" />
+        <child link="right_wheel_link" />
+        <origin xyz="${-base_length / 4.0} ${-(base_width + wheel_length) / 2.0} 0" rpy="0 0 0" />
+        <axis xyz="0 1 0" />
     </joint>
     <joint name="base_left_wheel_joint" type="continuous">
-        <parent link="base_link"/>
-        <child link="left_wheel_link"/>
-        <origin xyz="${-base_length / 4.0} ${-(base_width+ wheel_length)/2.0} 0" rpy="0 0 0"/>
-        <axis xyz="0 1 0"/>
+        <parent link="base_link" />
+        <child link="left_wheel_link" />
+        <origin xyz="${-base_length / 4.0} ${(base_width + wheel_length) / 2.0} 0" rpy="0 0 0" />
+        <axis xyz="0 1 0" />
     </joint>
     <joint name="base_caster_wheel_joint" type="fixed">
-        <parent link="base_link"/>
-        <child link="caster_wheel_link"/>
-        <origin xyz="${base_length / 3.0} 0 ${-(base_height / 4)}" rpy="0 0 0"/>
-    </joint>
-    <joint name="base_footprint_joint" type="fixed">
-        <parent link="base_footprint"/>
-        <child link="base_link"/>
-        <origin xyz="0 0 ${base_height / 2.0}" rpy="0 0 0"/>
+        <parent link="base_link" />
+        <child link="caster_wheel_link" />
+        <origin xyz="${base_length / 3.0} 0 ${-wheel_radius / 2.0}" rpy="0 0 0" />
     </joint>
 </robot>

Commit message: xacro add

File: ros2_ws/src/my_robot-description/urdf/robot-wheel.urdf.xacro (robot description, xacro)
@@ -16,5 +16,11 @@
             <material name="blue" />
         </visual>
-        <xacro:box-inertia m="5" l="${base_length}" w="${base_width}" h="${base_height}" xyz="0 0 ${base_height / 2.0}" rpy="0 0 0" />
+        <collision>
+            <geometry>
+                <box size="${base_length} ${base_width} ${base_height}" />
+            </geometry>
+            <origin xyz="0 0 ${base_height / 2.0}" rpy="0 0 0" />
+        </collision>
+        <!-- <xacro:box_inertia m="5" l="${base_length}" w="${base_width}" h="${base_height}" xyz="0 0 ${base_height / 2.0}" rpy="0 0 0" /> -->
     </link>
     <xacro:macro name="wheel_link" params="prefix">
@@ -27,4 +33,10 @@
                 <material name="grey" />
             </visual>
+            <collision>
+                <geometry>
+                    <cylinder radius="${wheel_radius}" length="${wheel_length}" />
+                </geometry>
+                <origin xyz="0 0 0" rpy="${pi / 2.0} 0 0" />
+            </collision>
         </link>
     </xacro:macro>
@@ -39,4 +51,10 @@
             <material name="grey" />
         </visual>
+        <collision>
+            <geometry>
+                <sphere radius="${wheel_radius / 2.0}" />
+            </geometry>
+            <origin xyz="0 0 0" rpy="0 0 0" />
+        </collision>
     </link>
     <joint name="base_joint" type="fixed">
