Commit message: fix spawn gazebo

File: ros2_ws/src/my_robot-description/urdf/common_properties.xacro (robot description, xacro)
@@ -7,11 +7,29 @@
         <color rgba="0.5 0.5 0.5 1" />
     </material>
-    <xacro:macro name="box_inertia" params="m l h w xyz rpy">
+    <xacro:macro name="box_inertia" params="m l w h xyz rpy">
         <inertial>
-            <origin xyz="${xyz}" rpy="${rpy}"/>
-            <mass value="${m}"/>
+            <origin xyz="${xyz}" rpy="${rpy}" />
+            <mass value="${m}" />
             <inertia ixx="${(m/12) * (h*h + l*l)}" ixy="0" ixz="0"
-             iyy="{$(m/12) * (w*w + h*h)}" iyz="0"
-             izz="{$(m/12 * (w*w + l*l)}"/>
+                     iyy="${(m/12) * (w*w + l*l)}" iyz="0"
+                     izz="${(m/12) * (w*w + h*h)}" />
+        </inertial>
+    </xacro:macro>
+    <xacro:macro name="cylinder_inertia" params="m r h xyz rpy">
+        <inertial>
+            <origin xyz="${xyz}" rpy="${rpy}" />
+            <mass value="${m}" />
+            <inertia ixx="${(m/12) * (3*r*r + h*h)}" ixy="0" ixz="0"
+                     iyy="${(m/12) * (3*r*r + h*h)}" iyz="0"
+                     izz="${(m/2) * (r*r)}" />
+        </inertial>
+    </xacro:macro>
+    <xacro:macro name="sphere_inertia" params="m r xyz rpy">
+        <inertial>
+            <origin xyz="${xyz}" rpy="${rpy}" />
+            <mass value="${m}" />
+            <inertia ixx="${(2/5) * m * r * r}" ixy="0" ixz="0"
+                     iyy="${(2/5) * m * r * r}" iyz="0"
+                     izz="${(2/5) * m * r * r}" />
         </inertial>
     </xacro:macro>

File: ros2_ws/src/my_robot-description/urdf/robot-wheel.urdf.xacro (robot description, xacro)
@@ -22,5 +22,6 @@
             <origin xyz="0 0 ${base_height / 2.0}" rpy="0 0 0" />
         </collision>
-        <!-- <xacro:box_inertia m="5" l="${base_length}" w="${base_width}" h="${base_height}" xyz="0 0 ${base_height / 2.0}" rpy="0 0 0" /> -->
+        <xacro:box_inertia m="5.0" l="${base_length}" w="${base_width}" h="${base_height}"
+                           xyz="0 0 ${base_height / 2.0}" rpy="0 0 0" />
     </link>
     <xacro:macro name="wheel_link" params="prefix">
@@ -39,4 +40,6 @@
                 <origin xyz="0 0 0" rpy="${pi / 2.0} 0 0" />
             </collision>
+            <xacro:cylinder_inertia m="1.0" r="${wheel_radius}" h="${wheel_length}"
+                                    xyz="0 0 0" rpy="${pi / 2.0} 0 0" />
         </link>
     </xacro:macro>
@@ -57,4 +60,6 @@
             <origin xyz="0 0 0" rpy="0 0 0" />
         </collision>
+        <xacro:sphere_inertia m="0.5" r="${wheel_radius / 2.0}"
+                              xyz="0 0 0" rpy="0 0 0" />
     </link>
     <joint name="base_joint" type="fixed">
