Commit message: fix all

File: ros2_ws/src/my_robot-description/urdf/mobile_base_gazebo.xacro (robot description, xacro)
@@ -6,3 +6,37 @@
      </material>
  </gazebo>
+ <gazebo reference="right_wheel_link">
+    <material>
+       Gazebo/Grey
+    </material>
+</gazebo>
+<gazebo reference="left_wheel_link">
+    <material>
+       Gazebo/Grey
+    </material>
+</gazebo>
+<gazebo reference="caster_wheel_link">
+    <material>
+       Gazebo/Grey
+    </material>
+</gazebo>
+<gazebo>
+    <plugin name="diff_drive_contorller" filename="libgazebo_ros_diff_drive.so">
+        <!-- Update rate in Hz -->
+        <update_rate>50</update_rate>
+        <!-- wheels -->
+        <left_joint>base_left_wheel_joint</left_joint>
+        <right_joint>rbase_ight_wheel_joint</right_joint>
+        <!-- kinematics -->
+        <wheel_separation>0.45</wheel_separation>
+        <wheel_diameter>0.2</wheel_diameter>
+        <!-- output -->
+        <publish_odom>true</publish_odom>
+        <publish_odom_tf>true</publish_odom_tf>
+        <publish_wheel_tf>true</publish_wheel_tf>
+        <odometry_topic>odom</odometry_topic>
+        <odometry_frame>odom</odometry_frame>
+        <robot_base_frame>base_footprint</robot_base_frame>
+      </plugin>
+</gazebo>
 </robot>
